File: TrainingRecruitmentFlyer.kicad_pcb (KiCad board)
At the start: 2 copper layers, 59.7 x 95.5 mm, 188 parts, among them SW1 3P1T_Fused, U1 VNH5019A-E, U10 LS_4, U2 VNH5019A-E, U3 3.3V_OKI, U4 LS_1, U5 LS_2, U6 TM4C129E_Launchpad_X9, U7 Picoblade-3, U8 Picoblade-3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

Commit message: Fixed Van's email
Other:
- board text added: "Questions? Contact Marsrover@mst.edu, Jacob Lipina (jrlwd5@mst.edu), or Andrew Van Horn (asvdgv@mst.edu)"
- board text removed: "Questions? Contact Marsrover@mst.edu, Jacob Lipina (jrlwd5@mst.edu), or Andrew Van Horn (asvgdv@mst.edu)"
Changed lines of the file:
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@@
     (effects (font (size 5 2.5) (thickness 0.3)))
   )
-  (gr_text "Questions? Contact Marsrover@mst.edu,\nJacob Lipina (jrlwd5@mst.edu), or\nAndrew Van Horn (asvgdv@mst.edu)" (at 155.702 230.251) (layer F.SilkS)
+  (gr_text "Questions? Contact Marsrover@mst.edu,\nJacob Lipina (jrlwd5@mst.edu), or\nAndrew Van Horn (asvdgv@mst.edu)" (at 155.702 230.251) (layer F.SilkS)
     (effects (font (size 1.14 1.4) (thickness 0.275)))
   )
